File: Arachnid_SOM/RK3328.kicad_sch (KiCad schematic)
At the start: 5 parts, among them Y1 24MHz

Commit message: First revision
Parts:
- added C71, C94: 100nf, Capacitor_SMD:C_0402_1005Metric, symbol Device:C
- added D2: D_TVS, Diode_SMD:D_SOD-882, symbol Device:D_TVS
- added R18: 133R, Resistor_SMD:R_0402_1005Metric, symbol Device:R
- added R19, R7: 2K, Resistor_SMD:R_0402_1005Metric, symbol Device:R
- added R21: 6.49K, Resistor_SMD:R_0402_1005Metric, symbol Device:R
- added R25, R26: 10K, Resistor_SMD:R_0402_1005Metric, symbol Device:R
- added R27, R6: 22R, Resistor_SMD:R_0402_1005Metric, symbol Device:R
- added SW1, SW2: SW_SPST, Button_Switch_SMD:SW_Push_1P1T_NO_Vertical_Wuerth_434133025816, symbol Switch:SW_SPST
Connections:
- net GND: now also J1.B10, J1.B11, J1.B7, J1.B8, J1.B9, C71.2, C94.2, D2.1 (A1), R18.2, R19.2, R21.2, R27.1, R7.2, SW1.2 (B)
- net USB0_DN: now also J1.A22
- net USB0_DP: now also J1.A23
- net USB1_DN: now also J1.A24
- net USB1_DP: now also J1.A25
- net VCC_IO: now also U1.J6 (USB30_AVDD_3V3), U1.K7 (USB30_VBUS), U1.T6 (USB20_VBUS)
- net at U1.G5 (USB30_EXTR): now also R7.1
- net USB30_TXN: now reaches U1.H2 (USB30_TXN)
- net USB30_TXN: now also J1.A18
- net USB30_TXP: now reaches U1.H3 (USB30_TXP)
- net USB30_TXP: now also J1.A19
- net USB30_RXP: now reaches U1.J2 (USB30_RXP)
- net USB30_RXP: now also J1.A17
- net USB30_RXN: now reaches U1.J3 (USB30_RXN)
- net USB30_RXN: now also J1.A16
- net LDO1 1.8V: now reaches U1.J5 (USB30_AVDD_1V8)
- net LDO1 1.8V: now also U1.P6 (HDMI_AVDD_1V8), U1.U5 (USB20_AVDD_1V8), U1.U6 (FEPHY_AVDD_1V8), R25.2, R26.2
- net LDO3 1.0V: now reaches U1.J7 (USB30_DVDD_1V0)
- net LDO3 1.0V: now also U1.M6 (HDMI_AVDD_1V0), U1.V5 (USB20_DVDD_1V0), U1.V6 (FEPHY_AVDD_1V0)
- net USB30_DP: now reaches U1.K1 (USB30_DP)
- net USB30_DP: now also J1.A21
- net USB30_DN: now reaches U1.K2 (USB30_DM)
- net USB30_DN: now also J1.A20
- net at U1.M4 (HDMI_EXTRES): now also R19.1
- net at U1.V7 (FEPHY_EXTRES): now also R21.1
- net at U1.W6 (USB20_EXTR): now also R18.1
- net RESET: now reaches U1.P21 (NPOR)
- net RESET: now also C71.1, R6.1
- net UART_SOM_RX: now reaches J1.A1
- net UART_SOM_RX: now also U1.Y15 (UART0_RX)
- net UART_SOM_TX: now reaches J1.A2
- net UART_SOM_TX: now also U1.AA15 (UART0_TX)
- net SD CD: now reaches J1.A26
- net SD CD: now also U1.V10 (SDMMC0_DETN)
- net SD D2: now reaches J1.A27
- net SD D2: now also U1.W13 (SDMMC0_D2)
- net SD D3: now reaches J1.A28
- net SD D3: now also U1.AA13 (SDMMC0_D3)
- net SD CMD: now reaches J1.A29
- net SD CMD: now also U1.Y13 (SDMMC0_CMD)
- net SD CLK: now reaches J1.A30
- net SD CLK: now also U1.W12 (SDMMC0_CLK)
- net SD D0: now reaches J1.A31
- net SD D0: now also U1.U10 (SDMMC0_D0)
- net SD D1: now reaches J1.A32
- net SD D1: now also U1.W11 (SDMMC0_D1)
- net +5V: now reaches J1.B1
- net +5V: now also J1.B2, J1.B3, J1.B4, J1.B5, J1.B6
- new net: R27.2, SW2.1 (A)
- new net: D2.2 (A2), R6.2, SW1.1 (A)
- new net SARADC_IN0: C94.1, R26.1, SW2.2 (B), U1.M18 (SARADC_IN0)
- new net SARADC_IN1: R25.1, U1.M17 (SARADC_IN1)
Other:
- moved on the sheet: C69, C70, Y1
