File: Arachnid_SOM/SOM Power.kicad_sch (KiCad schematic)
At the start: 40 parts

Commit message: First revision
Parts:
- added C72, C73, C74, C78, C79, C80, C81, C82, C83, C84, C86, C88: 100nf, Capacitor_SMD:C_0402_1005Metric, symbol Device:C
- added C75, C76: 4.7uf, Capacitor_SMD:C_0603_1608Metric, symbol Device:C
- added C77: 4.7uf, Capacitor_SMD:C_0402_1005Metric, symbol Device:C
- added C85, C87: 100nf, Capacitor_SMD:C_0402_1005Metric_Pad0.74x0.62mm_HandSolder, symbol Device:C
- added D14: LED, LED_SMD:LED_0603_1608Metric, symbol Device:LED
- added R20: 240R, Resistor_SMD:R_0402_1005Metric, symbol Device:R
- added R22, R23: 100R, Resistor_SMD:R_0402_1005Metric, symbol Device:R
- C7: footprint Capacitor_SMD:C_0603_1608Metric -> Capacitor_SMD:C_0402_1005Metric_Pad0.74x0.62mm_HandSolder
Connections:
- net GND: now also C31.2, U1.R4 (CODEC_AVSS), U2.21 (REFGND), C72.2, C73.2, C74.2, C75.2, C76.2, C77.2, C78.2, C79.2, C80.2, C81.2, C82.2, C83.2, C84.2, C85.2, C86.2, C87.2, C88.2
- net LDO1 1.8V: now also U1.H5 (PLL_AVDD_1V8), U1.H6 (VCCIO6), U1.K6 (VCCIO_PMU), U1.M16 (SARADC_AVDD_1V8), U1.N16 (OTP_VCC_1V8), U1.N5 (CODEC_AVDD_1V8), U1.N6 (VDAC_AVDD_1V8), U1.R16 (VCCIO5), U1.T7 (VCCIO1), U1.U12 (VCCIO4), U1.U7 (VCCIO3), C74.1, C76.1, C77.1, C78.1, C79.1, C80.1, C81.1, C82.1, C83.1, C84.1, C87.1, C88.1
- net LDO2 1.8V: now also U1.T17 (VCCIO2), C86.1
- net LDO3 1.0V: now also U1.H7 (PLL_DVDD_1V0), U1.M5 (VDD_PMU), C73.1, C75.1, C85.1
- net OUT1: now also D14.1 (K)
- net VCC_IO: now also R20.1
- net VDD Core: now also R22.1, R22.2
- net VDD Logic: now also R23.1, R23.2
- net 32KOUT: now reaches U2.25 (CLK32K)
- net at U2.32 (PWRON): now also C72.1
- new net: D14.2 (A), R20.2
Other:
- note added: ">12mil (close)"
- note added: "close"
- moved on the sheet: C1, C10, C11, C12, C13, C14, C15, C16, C17, C18, C19, C2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
