File: Arachnid_SOM/SOM_DDR3.kicad_sch (KiCad schematic)
At the start: 49 parts, among them U3 AS4C256M16D3, U4 AS4C256M16D3

Commit message: First revision
Parts:
- added C89, C90, C93: 100nf, Capacitor_SMD:C_0402_1005Metric, symbol Device:C
- added C91, C92: 10nf, Capacitor_SMD:C_0402_1005Metric, symbol Device:C
- added R13, R14, R15, R16, R17: 56R, Resistor_SMD:R_Array_Convex_4x0402, symbol R_Array:R_Array_4x
- added R24: 56R, Resistor_SMD:R_0402_1005Metric, symbol Device:R
- added TP1, TP2: TestPoint_Small, TestPoint:TestPoint_Pad_D1.5mm, symbol Connector:TestPoint_Small
- C33, C34, C36: footprint Capacitor_SMD:C_0603_1608Metric -> Capacitor_SMD:C_0402_1005Metric
Connections:
- net DDR3_A0: now also R16.3
- net DDR3_A1: now also R14.2
- net DDR3_A10: now also R8.4
- net DDR3_A11: now also R15.2
- net DDR3_A12: now also R14.1
- net DDR3_A13: now also R17.3
- net DDR3_A14: now also R15.4
- net DDR3_A2: now also R17.1
- net DDR3_A3: now also R16.2
- net DDR3_A4: now also R14.4
- net DDR3_A5: now also R16.4
- net DDR3_A6: now also R15.1
- net DDR3_A7: now also R17.4
- net DDR3_A8: now also R15.3
- net DDR3_A9: now also R17.2
- net DDR3_BA0: now also R13.4
- net DDR3_BA1: now also R14.3
- net DDR3_BA2: now also R16.1
- net DDR3_CASn: now also R13.1
- net DDR3_CKE: now also R8.3
- net DDR3_CLK_N: now also R8.2; no longer R4.2, U1.A20 (DDR3_CLK_N)
- net DDR3_CLK_P: now also R8.1; no longer R4.1, U1.B20 (DDR3_CLK_P)
- net DDR3_CSN0: now also R13.2
- net DDR3_RASn: now also R24.1
- net DDR3_WEn: now also R13.3
- net GND: now also C30.2, C32.2, C33.2, C34.2, C35.2, C36.2, C37.2, R11.2, U6.11 (PAD), U6.8 (GND), C89.2, C90.2, C91.2, C92.2, C93.2; no longer C37.1, R10.2, R11.1, U6.1 (REFIN)
- net PGOOD: now also TP1.1
- net VCC_DDR: now also C30.1, C33.1, C34.1, C35.1, C36.1, C93.1
- net VCC_IO: now also C32.1, U6.7 (EN), C90.1
- net VTT: now also R8.5, R8.6, R8.7, R8.8, R13.5, R13.6, R13.7, R13.8, R14.5, R14.6, R14.7, R14.8, R15.5, R15.6, R15.7, R15.8, R16.5, R16.6, R16.7, R16.8, R17.5, R17.6, R17.7, R17.8, R24.2
- net REFOUT: now reaches U3.H1 (VREFDQ)
- net REFOUT: now also U3.M8 (VREFCA), U4.H1 (VREFDQ), U4.M8 (VREFCA), U6.6 (REFOUT), C89.1, C91.1, C92.1, TP2.1
- new net: C37.1, R10.2, R11.1, U6.1 (REFIN)
- new net __DDR3_CLK_N: R4.2, U1.A20 (DDR3_CLK_N)
- new net __DDR3_CLK_P: R4.1, U1.B20 (DDR3_CLK_P)
Other:
- note added: "Near SOC"
- moved on the sheet: C30, C32, C33, C35, C38, C39, C40, C41, C42, C43, C44, C45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
