File: Arachnid_SOM/Arachnid_SOM.kicad_pcb (KiCad board)
At the start: 6 copper layers, 39.4 x 49.1 mm, 97 parts, among them U3 AS4C256M16D3, U4 AS4C256M16D3, Y1 24MHz

Commit message: First revision
Parts:
- removed the R8 at (128.3, 73.2)
- removed the R8 at (135.6, 68.4)
- removed the R8 at (128.3, 75.7)
- removed the R8 at (138.2, 68.4)
- removed the R8 at (128.3, 78.2)
- removed the R8 at (133.1, 68.4)
- added C71: 100nf, Capacitor_SMD:C_0402_1005Metric, F.Cu at (151.3, 109.3)
- added C72: 100nf, Capacitor_SMD:C_0402_1005Metric, F.Cu at (121.0, 101.3)
- added C73: 100nf, Capacitor_SMD:C_0402_1005Metric, B.Cu at (141.2, 93.0)
- added C74: 100nf, Capacitor_SMD:C_0402_1005Metric, F.Cu at (134.8, 89.0)
- added C75: 4.7uf, Capacitor_SMD:C_0603_1608Metric, F.Cu at (134.2, 91.8)
- added C76: 4.7uf, Capacitor_SMD:C_0603_1608Metric, F.Cu at (134.2, 90.3)
- added C77: 4.7uf, Capacitor_SMD:C_0402_1005Metric, F.Cu at (144.4, 103.5)
- added C78: 100nf, Capacitor_SMD:C_0402_1005Metric, B.Cu at (139.3, 94.3)
- added C79: 100nf, Capacitor_SMD:C_0402_1005Metric, B.Cu at (140.6, 97.8)
- added C80: 100nf, Capacitor_SMD:C_0402_1005Metric, F.Cu at (151.9, 95.8)
- added C81: 100nf, Capacitor_SMD:C_0402_1005Metric, F.Cu at (151.9, 94.8)
- added C82: 100nf, Capacitor_SMD:C_0402_1005Metric, F.Cu at (145.5, 103.5)
- added C83: 100nf, Capacitor_SMD:C_0402_1005Metric, F.Cu at (149.8, 103.5)
- added C84: 100nf, Capacitor_SMD:C_0402_1005Metric, B.Cu at (139.8, 92.5)
- added C85: 100nf, Capacitor_SMD:C_0402_1005Metric_Pad0.74x0.62mm_HandSolder, B.Cu at (139.1, 99.5)
- added C86: 100nf, Capacitor_SMD:C_0402_1005Metric, F.Cu at (151.9, 96.8)
- added C87: 100nf, Capacitor_SMD:C_0402_1005Metric_Pad0.74x0.62mm_HandSolder, B.Cu at (146.7, 95.6)
- added C88: 100nf, Capacitor_SMD:C_0402_1005Metric, B.Cu at (140.2, 96.2)
- added C89: 100nf, Capacitor_SMD:C_0402_1005Metric, F.Cu at (126.6, 79.6)
- added C90: 100nf, Capacitor_SMD:C_0402_1005Metric, F.Cu at (124.8, 78.0)
- added C91: 10nf, Capacitor_SMD:C_0402_1005Metric, B.Cu at (133.5, 74.4)
- added C92: 10nf, Capacitor_SMD:C_0402_1005Metric, B.Cu at (153.6, 78.5)
- added C93: 100nf, Capacitor_SMD:C_0402_1005Metric, B.Cu at (143.7, 92.6)
- added C94: 100nf, Capacitor_SMD:C_0402_1005Metric, F.Cu at (156.8, 100.2)
- added D14: LED, LED_SMD:LED_0603_1608Metric, F.Cu at (131.9, 104.9)
- added D2: D_TVS, Diode_SMD:D_SOD-882, F.Cu at (158.4, 106.7)
- added R13: 56R, Resistor_SMD:R_Array_Convex_4x0402, F.Cu at (129.8, 79.0)
- added R14: 56R, Resistor_SMD:R_Array_Convex_4x0402, F.Cu at (129.7, 72.5)
- added R15: 56R, Resistor_SMD:R_Array_Convex_4x0402, F.Cu at (131.2, 68.6)
- added R16: 56R, Resistor_SMD:R_Array_Convex_4x0402, F.Cu at (133.8, 68.6)
- added R17: 56R, Resistor_SMD:R_Array_Convex_4x0402, F.Cu at (136.4, 68.6)
- added R18: 133R, Resistor_SMD:R_0402_1005Metric, F.Cu at (140.3, 105.7)
- added R19: 2K, Resistor_SMD:R_0402_1005Metric, F.Cu at (134.8, 94.3)
- added R20: 240R, Resistor_SMD:R_0402_1005Metric, F.Cu at (132.1, 107.0)
- added R21: 6.49K, Resistor_SMD:R_0402_1005Metric, F.Cu at (140.3, 103.5)
- added R22: 100R, Resistor_SMD:R_0402_1005Metric, F.Cu at (122.7, 103.0)
- added R23: 100R, Resistor_SMD:R_0402_1005Metric, F.Cu at (130.9, 102.9)
- added R24: 56R, Resistor_SMD:R_0402_1005Metric, F.Cu at (127.7, 79.6)
- added R25: 10K, Resistor_SMD:R_0402_1005Metric, F.Cu at (156.1, 96.3)
- added R26: 10K, Resistor_SMD:R_0402_1005Metric, F.Cu at (151.3, 101.8)
- added R27: 22R, Resistor_SMD:R_0402_1005Metric, F.Cu at (158.2, 103.6)
- added R6: 22R, Resistor_SMD:R_0402_1005Metric, F.Cu at (151.3, 106.8)
- added R7: 2K, Resistor_SMD:R_0402_1005Metric, F.Cu at (134.8, 93.1)
- added R8: 56R, Resistor_SMD:R_Array_Convex_4x0402, F.Cu at (129.8, 76.3)
- added REF**: MountingHole_3.2mm_M3_DIN965_Pad, MountingHole:MountingHole_3.2mm_M3_DIN965_Pad, F.Cu at (139.7, 65.2)
- added REF**: MountingHole_2.7mm_M2.5_ISO7380, MountingHole:MountingHole_2.7mm_M2.5_ISO7380, F.Cu at (122.5, 67.8)
- added REF**: MountingHole_2.7mm_M2.5_ISO7380, MountingHole:MountingHole_2.7mm_M2.5_ISO7380, F.Cu at (156.8, 67.8)
- added SW1: SW_SPST, Button_Switch_SMD:SW_Push_1P1T_NO_Vertical_Wuerth_434133025816, F.Cu at (154.8, 107.8)
- added SW2: SW_SPST, Button_Switch_SMD:SW_Push_1P1T_NO_Vertical_Wuerth_434133025816, F.Cu at (154.8, 102.7)
- added TP1: TestPoint_Small, TestPoint:TestPoint_Pad_D1.5mm, F.Cu at (121.4, 73.6)
- added TP2: TestPoint_Small, TestPoint:TestPoint_Pad_D1.5mm, F.Cu at (124.2, 73.6)
- C30, C35, C59, C60, C61, C62: moved to B.Cu
- C33, C34: footprint Capacitor_SMD:C_0603_1608Metric -> Capacitor_SMD:C_0402_1005Metric
- C36: footprint Capacitor_SMD:C_0603_1608Metric -> Capacitor_SMD:C_0402_1005Metric; moved to B.Cu
- C7: footprint Capacitor_SMD:C_0603_1608Metric -> Capacitor_SMD:C_0402_1005Metric_Pad0.74x0.62mm_HandSolder
- moved C12 83.2 mm to (134.6, 102.0), turned to 0 degrees
- moved C10 80.7 mm to (134.6, 103.0), turned to 0 degrees
- moved C14 64.0 mm to (148.5, 104.2)
- moved C13 63.0 mm to (146.9, 104.2)
- moved C34 57.6 mm to (154.7, 93.5)
- moved C36 48.5 mm to (145.3, 94.0), turned to 180 degrees
- moved C30 45.7 mm to (144.7, 92.6), turned to -90 degrees
- moved C68 45.2 mm to (127.0, 84.8)
- moved C33 45.2 mm to (154.7, 92.3)
- moved C67 45.0 mm to (127.0, 83.8)
- moved C66 44.7 mm to (127.0, 82.8)
- moved C57 41.8 mm to (143.0, 68.6), turned to 90 degrees
- moved C35 41.5 mm to (142.7, 92.6), turned to -90 degrees
- moved C56 41.2 mm to (142.0, 68.6), turned to 90 degrees
- moved C65 41.1 mm to (124.2, 84.7)
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Connections:
- C22 pad 1: /RK3328 SOM - DDR3 A/SOM Power/LDO1 1.8V -> /RK3328 SOM - DDR3 A/LDO1 1.8V
- C25 pad 1: /RK3328 SOM - DDR3 A/SOM Power/LDO2 1.8V -> /RK3328 SOM - DDR3 A/LDO2 1.8V
- C27 pad 1: /RK3328 SOM - DDR3 A/SOM Power/LDO3 1.0V -> /RK3328 SOM - DDR3 A/LDO3 1.0V
- C30 pad 1: unconnected-(C30-Pad1) -> /RK3328 SOM - DDR3 A/VCC_DDR
- C30 pad 2: unconnected-(C30-Pad2) -> GND
- C31 pad 2: unconnected-(C31-Pad2) -> GND
- C32 pad 1: unconnected-(C32-Pad1) -> /RK3328 SOM - DDR3 A/VCC_IO
- C32 pad 2: unconnected-(C32-Pad2) -> GND
- C33 pad 1: unconnected-(C33-Pad1) -> /RK3328 SOM - DDR3 A/VCC_DDR
- C33 pad 2: unconnected-(C33-Pad2) -> GND
- C34 pad 1: unconnected-(C34-Pad1) -> /RK3328 SOM - DDR3 A/VCC_DDR
- C34 pad 2: unconnected-(C34-Pad2) -> GND
- C35 pad 1: unconnected-(C35-Pad1) -> /RK3328 SOM - DDR3 A/VCC_DDR
- C35 pad 2: unconnected-(C35-Pad2) -> GND
- C36 pad 1: unconnected-(C36-Pad1) -> /RK3328 SOM - DDR3 A/VCC_DDR
- C36 pad 2: unconnected-(C36-Pad2) -> GND
- C37 pad 1: GND -> Net-(U6-REFIN)
- C37 pad 2: Net-(C37-Pad2) -> GND
- J1 pad A1: unconnected-(J1-PadA1) -> /RK3328 SOM - DDR3 A/UART_SOM_RX
- J1 pad A16: unconnected-(J1-PadA16) -> /RK3328 SOM - DDR3 A/USB30_RXN
- J1 pad A17: unconnected-(J1-PadA17) -> /RK3328 SOM - DDR3 A/USB30_RXP
- J1 pad A18: unconnected-(J1-PadA18) -> /RK3328 SOM - DDR3 A/USB30_TXN
- J1 pad A19: unconnected-(J1-PadA19) -> /RK3328 SOM - DDR3 A/USB30_TXP
- J1 pad A2: unconnected-(J1-PadA2) -> /RK3328 SOM - DDR3 A/UART_SOM_TX
- J1 pad A20: unconnected-(J1-PadA20) -> /RK3328 SOM - DDR3 A/USB30_DN
- J1 pad A21: unconnected-(J1-PadA21) -> /RK3328 SOM - DDR3 A/USB30_DP
- J1 pad A22: unconnected-(J1-PadA22) -> /RK3328 SOM - DDR3 A/USB0_DN
- J1 pad A23: unconnected-(J1-PadA23) -> /RK3328 SOM - DDR3 A/USB0_DP
- J1 pad A24: unconnected-(J1-PadA24) -> /RK3328 SOM - DDR3 A/USB1_DN
- J1 pad A25: unconnected-(J1-PadA25) -> /RK3328 SOM - DDR3 A/USB1_DP
- J1 pad A26: unconnected-(J1-PadA26) -> /RK3328 SOM - DDR3 A/SD CD
- J1 pad A27: unconnected-(J1-PadA27) -> /RK3328 SOM - DDR3 A/SD D2
- J1 pad A28: unconnected-(J1-PadA28) -> /RK3328 SOM - DDR3 A/SD D3
- J1 pad A29: unconnected-(J1-PadA29) -> /RK3328 SOM - DDR3 A/SD CMD
- J1 pad A30: unconnected-(J1-PadA30) -> /RK3328 SOM - DDR3 A/SD CLK
- J1 pad A31: unconnected-(J1-PadA31) -> /RK3328 SOM - DDR3 A/SD D0
- J1 pad A32: unconnected-(J1-PadA32) -> /RK3328 SOM - DDR3 A/SD D1
- J1 pad B1: unconnected-(J1-PadB1) -> +5V
- J1 pad B10: unconnected-(J1-PadB10) -> GND
- J1 pad B11: unconnected-(J1-PadB11) -> GND
- J1 pad B2: unconnected-(J1-PadB2) -> +5V
- J1 pad B3: unconnected-(J1-PadB3) -> +5V
- J1 pad B4: unconnected-(J1-PadB4) -> +5V
- J1 pad B5: unconnected-(J1-PadB5) -> +5V
- J1 pad B6: unconnected-(J1-PadB6) -> +5V
- J1 pad B7: unconnected-(J1-PadB7) -> GND
- J1 pad B8: unconnected-(J1-PadB8) -> GND
- J1 pad B9: unconnected-(J1-PadB9) -> GND
- R10 pad 2: GND -> Net-(U6-REFIN)
- R11 pad 1: GND -> Net-(U6-REFIN)
- R11 pad 2: Net-(C37-Pad2) -> GND
- R4 pad 1: /RK3328 SOM - DDR3 A/SOM DDR3/DDR3_CLK_P -> /RK3328 SOM - DDR3 A/SOM DDR3/__DDR3_CLK_P
- R4 pad 2: /RK3328 SOM - DDR3 A/SOM DDR3/DDR3_CLK_N -> /RK3328 SOM - DDR3 A/SOM DDR3/__DDR3_CLK_N
- U1 pad A20: /RK3328 SOM - DDR3 A/SOM DDR3/DDR3_CLK_N -> /RK3328 SOM - DDR3 A/SOM DDR3/__DDR3_CLK_N
- U1 pad AA13: (no net) -> /RK3328 SOM - DDR3 A/SD D3
- U1 pad AA15: (no net) -> /RK3328 SOM - DDR3 A/UART_SOM_TX
- U1 pad B20: /RK3328 SOM - DDR3 A/SOM DDR3/DDR3_CLK_P -> /RK3328 SOM - DDR3 A/SOM DDR3/__DDR3_CLK_P
- U1 pad G5: unconnected-(U1D-USB30_EXTR-PadG5) -> Net-(U1D-USB30_EXTR)
- U1 pad H2: unconnected-(U1D-USB30_TXN-PadH2) -> /RK3328 SOM - DDR3 A/USB30_TXN
- U1 pad H3: unconnected-(U1D-USB30_TXP-PadH3) -> /RK3328 SOM - DDR3 A/USB30_TXP
- U1 pad H5: (no net) -> /RK3328 SOM - DDR3 A/LDO1 1.8V
- U1 pad H6: (no net) -> /RK3328 SOM - DDR3 A/LDO1 1.8V
- U1 pad H7: (no net) -> /RK3328 SOM - DDR3 A/LDO3 1.0V
- U1 pad J2: unconnected-(U1D-USB30_RXP-PadJ2) -> /RK3328 SOM - DDR3 A/USB30_RXP
- U1 pad J3: unconnected-(U1D-USB30_RXN-PadJ3) -> /RK3328 SOM - DDR3 A/USB30_RXN
- U1 pad J5: unconnected-(U1D-USB30_AVDD_1V8-PadJ5) -> /RK3328 SOM - DDR3 A/LDO1 1.8V
- U1 pad J6: unconnected-(U1D-USB30_AVDD_3V3-PadJ6) -> /RK3328 SOM - DDR3 A/VCC_IO
- U1 pad J7: unconnected-(U1D-USB30_DVDD_1V0-PadJ7) -> /RK3328 SOM - DDR3 A/LDO3 1.0V
- U1 pad K1: unconnected-(U1D-USB30_DP-PadK1) -> /RK3328 SOM - DDR3 A/USB30_DP
- U1 pad K2: unconnected-(U1D-USB30_DM-PadK2) -> /RK3328 SOM - DDR3 A/USB30_DN
- U1 pad K6: (no net) -> /RK3328 SOM - DDR3 A/LDO1 1.8V
- U1 pad K7: unconnected-(U1D-USB30_VBUS-PadK7) -> /RK3328 SOM - DDR3 A/VCC_IO
- U1 pad M16: (no net) -> /RK3328 SOM - DDR3 A/LDO1 1.8V
- U1 pad M17: (no net) -> /RK3328 SOM - DDR3 A/SARADC_IN1
- U1 pad M18: (no net) -> /RK3328 SOM - DDR3 A/SARADC_IN0
- U1 pad M4: unconnected-(U1D-HDMI_EXTRES-PadM4) -> Net-(U1D-HDMI_EXTRES)
- U1 pad M5: (no net) -> /RK3328 SOM - DDR3 A/LDO3 1.0V
- U1 pad M6: unconnected-(U1D-HDMI_AVDD_1V0-PadM6) -> /RK3328 SOM - DDR3 A/LDO3 1.0V
- U1 pad N16: (no net) -> /RK3328 SOM - DDR3 A/LDO1 1.8V
- U1 pad N5: (no net) -> /RK3328 SOM - DDR3 A/LDO1 1.8V
- U1 pad N6: (no net) -> /RK3328 SOM - DDR3 A/LDO1 1.8V
- U1 pad P21: unconnected-(U1E-NPOR-PadP21) -> /RK3328 SOM - DDR3 A/RESET
- U1 pad P6: unconnected-(U1D-HDMI_AVDD_1V8-PadP6) -> /RK3328 SOM - DDR3 A/LDO1 1.8V
- U1 pad R16: (no net) -> /RK3328 SOM - DDR3 A/LDO1 1.8V
- U1 pad R4: (no net) -> GND
- U1 pad T17: (no net) -> /RK3328 SOM - DDR3 A/LDO2 1.8V
- U1 pad T6: unconnected-(U1D-USB20_VBUS-PadT6) -> /RK3328 SOM - DDR3 A/VCC_IO
- U1 pad T7: (no net) -> /RK3328 SOM - DDR3 A/LDO1 1.8V
- U1 pad U10: (no net) -> /RK3328 SOM - DDR3 A/SD D0
- U1 pad U12: (no net) -> /RK3328 SOM - DDR3 A/LDO1 1.8V
- U1 pad U5: unconnected-(U1D-USB20_AVDD_1V8-PadU5) -> /RK3328 SOM - DDR3 A/LDO1 1.8V
- U1 pad U6: unconnected-(U1D-FEPHY_AVDD_1V8-PadU6) -> /RK3328 SOM - DDR3 A/LDO1 1.8V
- U1 pad U7: (no net) -> /RK3328 SOM - DDR3 A/LDO1 1.8V
- U1 pad V10: (no net) -> /RK3328 SOM - DDR3 A/SD CD
- U1 pad V5: unconnected-(U1D-USB20_DVDD_1V0-PadV5) -> /RK3328 SOM - DDR3 A/LDO3 1.0V
- U1 pad V6: unconnected-(U1D-FEPHY_AVDD_1V0-PadV6) -> /RK3328 SOM - DDR3 A/LDO3 1.0V
- U1 pad V7: unconnected-(U1D-FEPHY_EXTRES-PadV7) -> Net-(U1D-FEPHY_EXTRES)
- U1 pad W11: (no net) -> /RK3328 SOM - DDR3 A/SD D1
- U1 pad W12: (no net) -> /RK3328 SOM - DDR3 A/SD CLK
- U1 pad W13: (no net) -> /RK3328 SOM - DDR3 A/SD D2
- U1 pad W6: unconnected-(U1D-USB20_EXTR-PadW6) -> Net-(U1D-USB20_EXTR)
- U1 pad Y13: (no net) -> /RK3328 SOM - DDR3 A/SD CMD
- U1 pad Y15: (no net) -> /RK3328 SOM - DDR3 A/UART_SOM_RX
- U2 pad 21: unconnected-(U2-REFGND-Pad21) -> GND
- U2 pad 24: /RK3328 SOM - DDR3 A/SOM Power/LDO3 1.0V -> /RK3328 SOM - DDR3 A/LDO3 1.0V
- U2 pad 25: unconnected-(U2-CLK32K-Pad25) -> /RK3328 SOM - DDR3 A/SOM Power/32KOUT
- U2 pad 3: /RK3328 SOM - DDR3 A/SOM Power/LDO1 1.8V -> /RK3328 SOM - DDR3 A/LDO1 1.8V
- U2 pad 32: unconnected-(U2-PWRON-Pad32) -> Net-(U2-PWRON)
- U2 pad 5: /RK3328 SOM - DDR3 A/SOM Power/LDO2 1.8V -> /RK3328 SOM - DDR3 A/LDO2 1.8V
- U3 pad H1: unconnected-(U3-VREFDQ-PadH1) -> /RK3328 SOM - DDR3 A/SOM DDR3/REFOUT
- U3 pad M8: unconnected-(U3-VREFCA-PadM8) -> /RK3328 SOM - DDR3 A/SOM DDR3/REFOUT
- U4 pad H1: unconnected-(U4-VREFDQ-PadH1) -> /RK3328 SOM - DDR3 A/SOM DDR3/REFOUT
- U4 pad M8: unconnected-(U4-VREFCA-PadM8) -> /RK3328 SOM - DDR3 A/SOM DDR3/REFOUT
- U6 pad 1: GND -> Net-(U6-REFIN)
- U6 pad 11: (no net) -> GND
- U6 pad 6: unconnected-(U6-REFOUT-Pad6) -> /RK3328 SOM - DDR3 A/SOM DDR3/REFOUT
- U6 pad 7: unconnected-(U6-EN-Pad7) -> /RK3328 SOM - DDR3 A/VCC_IO
- U6 pad 8: unconnected-(U6-GND-Pad8) -> GND
Routing:
- net /RK3328 SOM - DDR3 A/SOM Power/VDD Core: track 0.00 -> 94.2 mm, vias 7 -> 16
- net /RK3328 SOM - DDR3 A/LDO1 1.8V: track 0.00 -> 84.0 mm, vias 0 -> 18
- net /RK3328 SOM - DDR3 A/VCC_IO: track 0.00 -> 73.0 mm, vias 0 -> 13
- net /RK3328 SOM - DDR3 A/SOM DDR3/REFOUT: track 0.00 -> 65.7 mm, vias 0 -> 6
- net GND: track 9.43 -> 69.3 mm, vias 190 -> 293
- net /RK3328 SOM - DDR3 A/LDO2 1.8V: track 0.00 -> 45.2 mm, vias 0 -> 4
- net /RK3328 SOM - DDR3 A/SOM Power/VDD Logic: track 0.00 -> 42.9 mm, vias 9 -> 21
- net /RK3328 SOM - DDR3 A/USB30_RXN: track 0.00 -> 36.7 mm, vias 0 -> 1
- net /RK3328 SOM - DDR3 A/USB30_RXP: track 0.00 -> 36.7 mm, vias 0 -> 1
- net /RK3328 SOM - DDR3 A/USB30_TXP: track 0.00 -> 36.6 mm, vias 0 -> 1
- net /RK3328 SOM - DDR3 A/USB30_TXN: track 0.00 -> 36.6 mm, vias 0 -> 1
- net /RK3328 SOM - DDR3 A/UART_SOM_RX: track 0.00 -> 33.7 mm, vias 0 -> 2
- net /RK3328 SOM - DDR3 A/UART_SOM_TX: track 0.00 -> 32.5 mm, vias 0 -> 2
- net /RK3328 SOM - DDR3 A/USB30_DN: track 0.00 -> 31.4 mm, vias 0 -> 1
- net /RK3328 SOM - DDR3 A/USB30_DP: track 0.00 -> 31.3 mm, vias 0 -> 1
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- added copper zone on B.Cu, net +5V
- added copper zone on F.Cu, net +5V
- added copper zone on In2.Cu, net +5V
- added copper zone on F.Cu, net /RK3328 SOM - DDR3 A/SOM DDR3/VTT
- added copper zone on B.Cu, net /RK3328 SOM - DDR3 A/SOM Power/VDD Core
- added copper zone on F.Cu, net /RK3328 SOM - DDR3 A/SOM Power/VDD Core
- added copper zone on In2.Cu, net /RK3328 SOM - DDR3 A/SOM Power/VDD Core
- added copper zone on B.Cu, net /RK3328 SOM - DDR3 A/SOM Power/VDD Logic
- added copper zone on F.Cu, net /RK3328 SOM - DDR3 A/SOM Power/VDD Logic
- added copper zone on In2.Cu, net /RK3328 SOM - DDR3 A/SOM Power/VDD Logic
- added copper zone on F.Cu, net /RK3328 SOM - DDR3 A/VCC_DDR
- added copper zone on F.Cu, net /RK3328 SOM - DDR3 A/VCC_IO
- added copper zone on In3.Cu, net /RK3328 SOM - DDR3 A/VCC_IO
- added copper zone on B.Cu, net GND
- added copper zone on F.Cu, net GND
- added copper zone on In3.Cu, net GND
- added copper zone on F.Cu, net Net-(U2-SW1)
- added copper zone on F.Cu, net Net-(U2-SW2)
- added copper zone on F.Cu, net Net-(U2-SW3)
- added copper zone on F.Cu, net Net-(U2-SW4)
Other:
- outline, holes or cut-outs redrawn
- board text added: "RK3328 SOM REV A0"
- board text added: "Recover"
- board text added: "Reset"

Commit message: Minor changes
Routing:
- net +5V: track 28.4 -> 37.2 mm
Other:
- board text added: "github.com/h3llf/RK3328_SOM"
Changed lines of the file:
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@@
 			)
 		)
-		(pad "1" thru_hole circle
+		(pad "" np_thru_hole circle
 			(at 0 0)
 			(size 5.6 5.6)
 			(drill 3.2)
-			(layers "*.Cu" "*.Mask")
-			(remove_unused_layers no)
+			(layers "F&B.Cu" "*.Mask")
 		)
 		(embedded_fonts no)
@@
 		)
 	)
+	(gr_text "github.com/h3llf/RK3328_SOM"
+		(at 151.8 112.55 0)
+		(layer "B.SilkS")
+		(effects
+			(font
+				(size 1 1)
+				(thickness 0.1)
+			)
+			(justify left bottom mirror)
+		)
+	)
 	(gr_text "6-layer JLC0616-3313 stackup\nUses via in pad extensively"
 		(at 210.825 22.3 0)
@@
 	)
 	(segment
+		(start 125.775 103.2)
+		(end 125.775 104.425)
+		(width 0.4)
+		(layer "B.Cu")
+		(net 4)
+	)
+	(segment
+		(start 124.779 106.079)
+		(end 125.4 106.7)
+		(width 0.4)
+		(layer "B.Cu")
+		(net 4)
+	)
+	(segment
+		(start 124.779 105.421)
+		(end 124.779 105.9)
+		(width 0.4)
+		(layer "B.Cu")
+		(net 4)
+	)
+	(segment
+		(start 126.6 104.8)
+		(end 126.899943 104.8)
+		(width 0.4)
+		(layer "B.Cu")
+		(net 4)
+	)
+	(segment
+		(start 127.601 106.049)
+		(end 126.75 106.9)
+		(width 0.4)
+		(layer "B.Cu")
+		(net 4)
+	)
+	(segment
+		(start 126.6 103.2)
+		(end 126.6 104.8)
+		(width 0.4)
+		(layer "B.Cu")
+		(net 4)
+	)
+	(segment
+		(start 125.775 104.425)
+		(end 125.75 104.45)
+		(width 0.4)
+		(layer "B.Cu")
+		(net 4)
+	)
+	(segment
+		(start 124.779 105.9)
+		(end 124.779 106.079)
+		(width 0.4)
+		(layer "B.Cu")
+		(net 4)
+	)
+	(segment
+		(start 126.899943 104.8)
+		(end 127.601 105.501057)
+		(width 0.4)
+		(layer "B.Cu")
+		(net 4)
+	)
+	(segment
+		(start 127.601 105.501057)
+		(end 127.601 106.049)
+		(width 0.4)
+		(layer "B.Cu")
+		(net 4)
+	)
+	(segment
+		(start 125.75 104.45)
+		(end 124.779 105.421)
+		(width 0.4)
+		(layer "B.Cu")
+		(net 4)
+	)
+	(segment
 		(start 123.895768 97.875)
 		(end 122.98 98.790768)
@@
 		(polygon
 			(pts
-				(xy 124.35 116.375) (xy 124.35 113.65) (xy 125.425 113.65) (xy 125.425 102.075) (xy 127.125 102.075)
+				(xy 124.35 116.375) (xy 124.35 113.65) (xy 125.075 113.65) (xy 125.075 102.075) (xy 127.125 102.075)
 				(xy 127.125 113.65) (xy 128 113.65) (xy 128 116.375)
 			)
